Commit message: complete disk stack urdf for testing

File: src/spm_sim_stack/spm_description/urdf/robots/spm_mechanism.urdf.xacro (robot description, xacro)
@@ -12,7 +12,8 @@
 	<xacro:property name="end_effector_mass" value="0.1"/>
 	<xacro:property name="probe_mass" value="0.05"/>
+	<xacro:property name="disk_offset" value="0.01"/>
 	<xacro:macro name="link_inertial" params="ixx iyy izz">
 		<inertial>
-			<origin xyz="0 0 0.0" rpy="0 0 0"/>
+			<origin xyz="0.0 0.0 0.0" rpy="0.0 0.0 0.0"/>
 			<mass value="${link_mass}"/>
 			<inertia
@@ -24,5 +25,5 @@
 	<xacro:macro name="disk_inertial" params="mass ixx iyy izz">
 		<inertial>
-			<origin xyz="0 0 0.0" rpy="0 0 0"/>
+			<origin xyz="0.0 0.0 0.0" rpy="0.0 0.0 0.0"/>
 			<mass value="${mass}"/>
 			<inertia
@@ -43,5 +44,5 @@
 		</gazebo>
 	</xacro:macro>
-	<xacro:macro name="spm_mechanism" params="base_link flange_link prefix *origin">
+	<xacro:macro name="spm_mechanism" params="base_link flange_link prefix base_x base_y base_z">
 	<!-- THESE FILES DO NOT EXIST YET -->
 	<!-- USE DETAILED STL/DAE FOR VISUAL, SIMPLIFIED STL FOR COLLISION -->
@@ -52,5 +53,5 @@
 					<mesh filename="file://$(find spm_description)/meshes/spm/visual/link_visual.dae"/>
 				</geometry>
-				<origin xyz="0.0 0 0" rpy="0 0 ${-pi/2}"/>
+				<origin xyz="0.0 0.0 0.0" rpy="0.0 0.0 0.0"/>
 			</visual>
 			<collision>
@@ -58,5 +59,5 @@
 					<mesh filename="file://$(find spm_description)/meshes/spm/visual/link_collision.stl"/>
 				</geometry>
-				<origin xyz="0.0 0 0" rpy="0 0 ${-pi/2}"/>
+				<origin xyz="0.0 0.0 0.0" rpy="0.0 0.0 0.0"/>
 			</collision>
 		</link>
@@ -67,5 +68,5 @@
 					<mesh filename="file://$(find spm_description)/meshes/spm/visual/link_visual.dae"/>
 				</geometry>
-				<origin xyz="0.0 0.1 0.1" rpy="0 0 ${-pi/2}"/>
+				<origin xyz="0.0 0.0 0.0" rpy="0.0 0.0 0.0"/>
 			</visual>
 			<collision>
@@ -73,5 +74,5 @@
 					<mesh filename="file://$(find spm_description)/meshes/spm/visual/link_collision.stl"/>
 				</geometry>
-				<origin xyz="0.0 0.1 0.1" rpy="0 0 ${-pi/2}"/>
+				<origin xyz="0.0 0.0 0.0" rpy="0.0 0.0 0.0"/>
 			</collision>
 		</link>
@@ -82,5 +83,5 @@
 					<mesh filename="file://$(find spm_description)/meshes/spm/visual/link_visual.dae"/>
 				</geometry>
-				<origin xyz="0.0 0.1 0" rpy="0 0 ${-pi/2}"/>
+				<origin xyz="0.0 0.0 0.0" rpy="0.0 0.0 0.0"/>
 			</visual>
 			<collision>
@@ -88,5 +89,5 @@
 					<mesh filename="file://$(find spm_description)/meshes/spm/visual/link_collision.stl"/>
 				</geometry>
-				<origin xyz="0.0 0.1 0" rpy="0 0 ${-pi/2}"/>
+				<origin xyz="0.0 0.0 0.0" rpy="0.0 0.0 0.0"/>
 			</collision>
 		</link>
@@ -105,5 +106,5 @@
 					<mesh filename="file://$(find spm_description)/meshes/spm/visual/disk1_visual.dae"/>
 				</geometry>
-				<origin xyz="0.0 0 0" rpy="0 0 0"/>
+				<origin xyz="0.0 0.0 0.0" rpy="0.0 0.0 0.0"/>
 			</visual>
 			<collision>
@@ -111,5 +112,5 @@
 					<mesh filename="file://$(find spm_description)/meshes/spm/visual/disk1_collision.stl"/>
 				</geometry>
-				<origin xyz="0.0 0 0" rpy="0 0 0"/>
+				<origin xyz="0.0 0.0 0.0" rpy="0.0 0.0 0.0"/>
 			</collision>
 		</link>
@@ -120,5 +121,5 @@
 					<mesh filename="file://$(find spm_description)/meshes/spm/visual/disk2_visual.dae"/>
 				</geometry>
-				<origin xyz="0.0 0 0" rpy="0 0 ${(2*pi)/3}"/>
+				<origin xyz="0.0 0.0 0.0" rpy="0.0 0.0 0.0"/>
 			</visual>
 			<collision>
@@ -126,5 +127,5 @@
 					<mesh filename="file://$(find spm_description)/meshes/spm/visual/disk2_collision.stl"/>
 				</geometry>
-				<origin xyz="0.0 0 0" rpy="0 0 ${(2*pi)/3}"/>
+				<origin xyz="0.0 0.0 0.0" rpy="0.0 0.0 0.0"/>
 			</collision>
 		</link>
@@ -135,5 +136,5 @@
 					<mesh filename="file://$(find spm_description)/meshes/spm/visual/disk3_visual.dae"/>
 				</geometry>
-				<origin xyz="0.0 0 0" rpy="0 0 ${(-1)*(2*pi)/3}"/>
+				<origin xyz="0.0 0.0 0.0" rpy="0.0 0.0 0.0"/>
 			</visual>
 			<collision>
@@ -141,5 +142,5 @@
 					<mesh filename="file://$(find spm_description)/meshes/spm/visual/disk3_collision.stl"/>
 				</geometry>
-				<origin xyz="0.0 0 0" rpy="0 0 ${(-1)*(2*pi)/3}"/>
+				<origin xyz="0.0 0.0 0.0" rpy="0.0 0.0 0.0"/>
 			</collision>
 		</link>
@@ -147,5 +148,5 @@
 		<link name="${prefix}end_effector">
 			<inertial>
-				<origin xyz="0 0 0.0" rpy="0 0 0"/>
+				<origin xyz="0.0 0.0 0.0" rpy="0.0 0.0 0.0"/>
 				<mass value="${end_effector_mass}"/>
 				<inertia
@@ -158,20 +159,38 @@
 					<mesh filename="file://$(find spm_description)/meshes/spm/visual/end_effector_visual.dae"/>
 				</geometry>
-				<origin xyz="0.0 0 0" rpy="0 0 0"/>
+				<origin xyz="0.0 0.0 0.0" rpy="0.0 0.0 0.0"/>
 			</visual>
 			<collision>
 				<geometry>
-					<mesh filename="file://$(find spm_description)/meshes/spm/visual/end_effector_visual.stl"/>
+					<mesh filename="file://$(find spm_description)/meshes/spm/visual/end_effector_collision.stl"/>
 				</geometry>
-				<origin xyz="0.0 0 0" rpy="0 0 0"/>
+				<origin xyz="0.0 0.0 0.0" rpy="0.0 0.0 0.0"/>
 			</collision>
 		</link>
 		<!-- BASE TO DISK JOINTS -->
 		<joint name="${prefix}disk1_to_base" type="continuous">
-			<axis xyz="0 0 1"/>
+			<axis xyz="0.0 0.0 1.0"/>
 			<limit effort="${joint_effort}" velocity="${joint_velocity}"/>
 			<parent link="${prefix}base_link"/>
 			<child link="${prefix}disk1"/>
-			<xacro:insert_block name="origin"/>
+			<origin xyz="${base_x} ${base_y} ${base_z+disk_offset}" rpy="0.0 0.0 0.0"/>
+			<dynamics damping="${joint_damping}" friction="${joint_friction}"/>
 		</joint>
+		<joint name="${prefix}disk2_to_base" type="continuous">
+			<axis xyz="0.0 0.0 1.0"/>
+			<limit effort="${joint_effort}" velocity="${joint_velocity}"/>
+			<parent link="${prefix}base_link"/>
+			<child link="${prefix}disk2"/>
+			<origin xyz="${base_x} ${base_y} ${base_z+(2*disk_offset)}" rpy="0.0 0.0 0.0"/>
+			<dynamics damping="${joint_damping}" friction="${joint_friction}"/>
+		</joint>
+		<joint name="${prefix}disk3_to_base" type="continuous">
+			<axis xyz="0.0 0.0 1.0"/>
+			<limit effort="${joint_effort}" velocity="${joint_velocity}"/>
+			<parent link="${prefix}base_link"/>
+			<child link="${prefix}disk3"/>
+			<origin xyz="${base_x} ${base_y} ${base_z+(3*disk_offset)}" rpy="0.0 0.0 0.0"/>
+			<dynamics damping="${joint_damping}" friction="${joint_friction}"/>
+		</joint>
+		<!-- DISK TO LINK JOINTS -->
 	</xacro:macro>

Commit message: add urdf assembly, functional launch using urdf_tutorial pkg

File: src/spm_sim_stack/spm_description/urdf/robots/spm_mechanism.urdf.xacro (robot description, xacro)
@@ -33,5 +33,5 @@
 		</inertial>
 	</xacro:macro>
-	<xacro:macro name="material_visual" params="ref_link ambient diffuse specular">
+	<xacro:macro name="material_collision" params="ref_link ambient diffuse specular">
 		<gazebo reference="${ref_link}">
 			<visual>
@@ -44,12 +44,12 @@
 		</gazebo>
 	</xacro:macro>
-	<xacro:macro name="spm_mechanism" params="base_link flange_link prefix base_x base_y base_z">
-	<!-- THESE FILES DO NOT EXIST YET -->
-	<!-- USE DETAILED STL/DAE FOR VISUAL, SIMPLIFIED STL FOR COLLISION -->
+	<xacro:macro name="spm_mechanism" params="base_link prefix base_x base_y base_z">
+	<!-- ONLY USING COLLISION MESHES FOR INITIAL TESTING -->
+	<!-- REMEMBER TO ADD VISUAL/COLLISION MESHES!!!!~
 		<link name="${prefix}link1">
 			<xacro:link_inertial ixx="0.0001" iyy="0.0001" izz="0.0001"/>
 			<visual>
 				<geometry>
-					<mesh filename="file://$(find spm_description)/meshes/spm/visual/link_visual.dae"/>
+					<mesh filename="file://$(find spm_description)/meshes/spm/visual/link_collision.stl"/>
 				</geometry>
 				<origin xyz="0.0 0.0 0.0" rpy="0.0 0.0 0.0"/>
@@ -66,5 +66,5 @@
 			<visual>
 				<geometry>
-					<mesh filename="file://$(find spm_description)/meshes/spm/visual/link_visual.dae"/>
+					<mesh filename="file://$(find spm_description)/meshes/spm/visual/link_collision.stl"/>
 				</geometry>
 				<origin xyz="0.0 0.0 0.0" rpy="0.0 0.0 0.0"/>
@@ -81,5 +81,5 @@
 			<visual>
 				<geometry>
-					<mesh filename="file://$(find spm_description)/meshes/spm/visual/link_visual.dae"/>
+					<mesh filename="file://$(find spm_description)/meshes/spm/visual/link_collision.stl"/>
 				</geometry>
 				<origin xyz="0.0 0.0 0.0" rpy="0.0 0.0 0.0"/>
@@ -92,4 +92,5 @@
 			</collision>
 		</link>
+		-->
 		<!-- DISK LINKS -->
 		<link name="base_link">
@@ -104,5 +105,5 @@
 			<visual>
 				<geometry>
-					<mesh filename="file://$(find spm_description)/meshes/spm/visual/disk1_visual.dae"/>
+					<mesh filename="file://$(find spm_description)/meshes/disk1_collision.stl"/>
 				</geometry>
 				<origin xyz="0.0 0.0 0.0" rpy="0.0 0.0 0.0"/>
@@ -110,5 +111,5 @@
 			<collision>
 				<geometry>
-					<mesh filename="file://$(find spm_description)/meshes/spm/visual/disk1_collision.stl"/>
+					<mesh filename="file://$(find spm_description)/meshes/disk1_collision.stl"/>
 				</geometry>
 				<origin xyz="0.0 0.0 0.0" rpy="0.0 0.0 0.0"/>
@@ -119,5 +120,5 @@
 			<visual>
 				<geometry>
-					<mesh filename="file://$(find spm_description)/meshes/spm/visual/disk2_visual.dae"/>
+					<mesh filename="file://$(find spm_description)/meshes/disk2_collision.stl"/>
 				</geometry>
 				<origin xyz="0.0 0.0 0.0" rpy="0.0 0.0 0.0"/>
@@ -125,5 +126,5 @@
 			<collision>
 				<geometry>
-					<mesh filename="file://$(find spm_description)/meshes/spm/visual/disk2_collision.stl"/>
+					<mesh filename="file://$(find spm_description)/meshes/disk2_collision.stl"/>
 				</geometry>
 				<origin xyz="0.0 0.0 0.0" rpy="0.0 0.0 0.0"/>
@@ -134,5 +135,5 @@
 			<visual>
 				<geometry>
-					<mesh filename="file://$(find spm_description)/meshes/spm/visual/disk3_visual.dae"/>
+					<mesh filename="file://$(find spm_description)/meshes/disk3_collision.stl"/>
 				</geometry>
 				<origin xyz="0.0 0.0 0.0" rpy="0.0 0.0 0.0"/>
@@ -140,10 +141,10 @@
 			<collision>
 				<geometry>
-					<mesh filename="file://$(find spm_description)/meshes/spm/visual/disk3_collision.stl"/>
+					<mesh filename="file://$(find spm_description)/meshes/disk3_collision.stl"/>
 				</geometry>
 				<origin xyz="0.0 0.0 0.0" rpy="0.0 0.0 0.0"/>
 			</collision>
 		</link>
-		<!-- END EFFECTOR -->
+		<!-- END EFFECTOR
 		<link name="${prefix}end_effector">
 			<inertial>
@@ -157,5 +158,5 @@
 			<visual>
 				<geometry>
-					<mesh filename="file://$(find spm_description)/meshes/spm/visual/end_effector_visual.dae"/>
+					<mesh filename="file://$(find spm_description)/meshes/spm/visual/end_effector_collision.stl"/>
 				</geometry>
 				<origin xyz="0.0 0.0 0.0" rpy="0.0 0.0 0.0"/>
@@ -168,4 +169,5 @@
 			</collision>
 		</link>
+		-->
 		<!-- BASE TO DISK JOINTS -->
 		<joint name="${prefix}disk1_to_base" type="continuous">
@@ -195,2 +197,3 @@
 		<!-- DISK TO LINK JOINTS -->
 	</xacro:macro>
+</robot>

Commit message: add disk+link urdf

File: src/spm_sim_stack/spm_description/urdf/robots/spm_mechanism.urdf.xacro (robot description, xacro)
@@ -12,5 +12,4 @@
 	<xacro:property name="end_effector_mass" value="0.1"/>
 	<xacro:property name="probe_mass" value="0.05"/>
-	<xacro:property name="disk_offset" value="0.01"/>
 	<xacro:macro name="link_inertial" params="ixx iyy izz">
 		<inertial>
@@ -46,16 +45,16 @@
 	<xacro:macro name="spm_mechanism" params="base_link prefix base_x base_y base_z">
 	<!-- ONLY USING COLLISION MESHES FOR INITIAL TESTING -->
-	<!-- REMEMBER TO ADD VISUAL/COLLISION MESHES!!!!~
+	<!-- REMEMBER TO ADD VISUAL/COLLISION MESHES!!!!~ -->
 		<link name="${prefix}link1">
 			<xacro:link_inertial ixx="0.0001" iyy="0.0001" izz="0.0001"/>
 			<visual>
 				<geometry>
-					<mesh filename="file://$(find spm_description)/meshes/spm/visual/link_collision.stl"/>
-				</geometry>
-				<origin xyz="0.0 0.0 0.0" rpy="0.0 0.0 0.0"/>
-			</visual>
-			<collision>
-				<geometry>
-					<mesh filename="file://$(find spm_description)/meshes/spm/visual/link_collision.stl"/>
+					<mesh filename="file://$(find spm_description)/meshes/link_collision.stl"/>
+				</geometry>
+				<origin xyz="0.0 0.0 0.0" rpy="0.0 0.0 0.0"/>
+			</visual>
+			<collision>
+				<geometry>
+					<mesh filename="file://$(find spm_description)/meshes/link_collision.stl"/>
 				</geometry>
 				<origin xyz="0.0 0.0 0.0" rpy="0.0 0.0 0.0"/>
@@ -66,11 +65,11 @@
 			<visual>
 				<geometry>
-					<mesh filename="file://$(find spm_description)/meshes/spm/visual/link_collision.stl"/>
-				</geometry>
-				<origin xyz="0.0 0.0 0.0" rpy="0.0 0.0 0.0"/>
-			</visual>
-			<collision>
-				<geometry>
-					<mesh filename="file://$(find spm_description)/meshes/spm/visual/link_collision.stl"/>
+					<mesh filename="file://$(find spm_description)/meshes/link_collision.stl"/>
+				</geometry>
+				<origin xyz="0.0 0.0 0.0" rpy="0.0 0.0 0.0"/>
+			</visual>
+			<collision>
+				<geometry>
+					<mesh filename="file://$(find spm_description)/meshes/link_collision.stl"/>
 				</geometry>
 				<origin xyz="0.0 0.0 0.0" rpy="0.0 0.0 0.0"/>
@@ -81,16 +80,15 @@
 			<visual>
 				<geometry>
-					<mesh filename="file://$(find spm_description)/meshes/spm/visual/link_collision.stl"/>
-				</geometry>
-				<origin xyz="0.0 0.0 0.0" rpy="0.0 0.0 0.0"/>
-			</visual>
-			<collision>
-				<geometry>
-					<mesh filename="file://$(find spm_description)/meshes/spm/visual/link_collision.stl"/>
-				</geometry>
-				<origin xyz="0.0 0.0 0.0" rpy="0.0 0.0 0.0"/>
-			</collision>
-		</link>
-		-->
+					<mesh filename="file://$(find spm_description)/meshes/link_collision.stl"/>
+				</geometry>
+				<origin xyz="0.0 0.0 0.0" rpy="0.0 0.0 0.0"/>
+			</visual>
+			<collision>
+				<geometry>
+					<mesh filename="file://$(find spm_description)/meshes/link_collision.stl"/>
+				</geometry>
+				<origin xyz="0.0 0.0 0.0" rpy="0.0 0.0 0.0"/>
+			</collision>
+		</link>
 		<!-- DISK LINKS -->
 		<link name="base_link">
@@ -158,11 +156,11 @@
 			<visual>
 				<geometry>
-					<mesh filename="file://$(find spm_description)/meshes/spm/visual/end_effector_collision.stl"/>
-				</geometry>
-				<origin xyz="0.0 0.0 0.0" rpy="0.0 0.0 0.0"/>
-			</visual>
-			<collision>
-				<geometry>
-					<mesh filename="file://$(find spm_description)/meshes/spm/visual/end_effector_collision.stl"/>
+					<mesh filename="file://$(find spm_description)/meshes/end_effector_collision.stl"/>
+				</geometry>
+				<origin xyz="0.0 0.0 0.0" rpy="0.0 0.0 0.0"/>
+			</visual>
+			<collision>
+				<geometry>
+					<mesh filename="file://$(find spm_description)/meshes/end_effector_collision.stl"/>
 				</geometry>
 				<origin xyz="0.0 0.0 0.0" rpy="0.0 0.0 0.0"/>
@@ -176,5 +174,5 @@
 			<parent link="${prefix}base_link"/>
 			<child link="${prefix}disk1"/>
-			<origin xyz="${base_x} ${base_y} ${base_z+disk_offset}" rpy="0.0 0.0 0.0"/>
+			<origin xyz="${base_x} ${base_y} ${base_z}" rpy="0.0 0.0 0.0"/>
 			<dynamics damping="${joint_damping}" friction="${joint_friction}"/>
 		</joint>
@@ -184,5 +182,5 @@
 			<parent link="${prefix}base_link"/>
 			<child link="${prefix}disk2"/>
-			<origin xyz="${base_x} ${base_y} ${base_z+(2*disk_offset)}" rpy="0.0 0.0 0.0"/>
+			<origin xyz="${base_x} ${base_y} ${base_z-0.00381}" rpy="0.0 0.0 0.0"/>
 			<dynamics damping="${joint_damping}" friction="${joint_friction}"/>
 		</joint>
@@ -192,8 +190,32 @@
 			<parent link="${prefix}base_link"/>
 			<child link="${prefix}disk3"/>
-			<origin xyz="${base_x} ${base_y} ${base_z+(3*disk_offset)}" rpy="0.0 0.0 0.0"/>
+			<origin xyz="${base_x} ${base_y} ${base_z+0.01143}" rpy="0.0 0.0 0.0"/>
 			<dynamics damping="${joint_damping}" friction="${joint_friction}"/>
 		</joint>
 		<!-- DISK TO LINK JOINTS -->
+		<joint name="${prefix}link1_to_disk1" type="continuous">
+			<axis xyz="0.0 0.0 1.0"/>
+			<limit effort="${joint_effort}" velocity="${joint_velocity}"/>
+			<parent link="${prefix}disk1"/>
+			<child link="${prefix}link1"/>
+			<origin xyz="0.0 0.060411 0.036634" rpy="${pi/4} 0.0 0.0"/>
+			<dynamics damping="${joint_damping}" friction="${joint_friction}"/>
+		</joint>
+		<joint name="${prefix}link2_to_disk2" type="continuous">
+			<axis xyz="0.0 0.0 1.0"/>
+			<limit effort="${joint_effort}" velocity="${joint_velocity}"/>
+			<parent link="${prefix}disk2"/>
+			<child link="${prefix}link2"/>
+			<origin xyz="0.052317 -0.030206 0.040444" rpy="${pi/4} 0.0 ${-2*pi/3}"/>
+			<dynamics damping="${joint_damping}" friction="${joint_friction}"/>
+		</joint>
+		<joint name="${prefix}link3_to_disk3" type="continuous">
+			<axis xyz="0.0 0.0 1.0"/>
+			<limit effort="${joint_effort}" velocity="${joint_velocity}"/>
+			<parent link="${prefix}disk3"/>
+			<child link="${prefix}link3"/>
+			<origin xyz="-0.052317 -0.030206 0.025204" rpy="${pi/4} 0.0 ${2*pi/3}"/>
+			<dynamics damping="${joint_damping}" friction="${joint_friction}"/>
+		</joint>
 	</xacro:macro>
 </robot>

Commit message: new link_collision.stl to fix default orientation

File: src/spm_sim_stack/spm_description/urdf/robots/spm_mechanism.urdf.xacro (robot description, xacro)
@@ -92,11 +92,5 @@
 		</link>
 		<!-- DISK LINKS -->
-		<link name="base_link">
-			<visual>
-				<geometry>
-					<box size="0.1 0.1 0.01"/>
-				</geometry>
-			</visual>
-		</link>
+		<link name="base_link"/>
 		<link name="${prefix}disk1">
 			<xacro:disk_inertial mass="${disk1_mass}" ixx="0.0001" iyy="0.0001" izz="0.0001"/>
@@ -218,4 +212,5 @@
 			<dynamics damping="${joint_damping}" friction="${joint_friction}"/>
 		</joint>
+		<!-- LINK TO END EFFECTOR JOINTS -->
 	</xacro:macro>
 </robot>

Commit message: add primary joint1 to end effector joint

File: src/spm_sim_stack/spm_description/urdf/robots/spm_mechanism.urdf.xacro (robot description, xacro)
@@ -2,6 +2,6 @@
 <robot xmlns:xacro="http://www.ros.org/wiki/xacro">
 	<!-- ALL VALUES ARE PLACEHOLDERS -->
-  <xacro:property name="joint_effort" value="3.0"/>
-  <xacro:property name="joint_velocity" value="6.28318"/>
+  	<xacro:property name="joint_effort" value="3.0"/>
+  	<xacro:property name="joint_velocity" value="6.28318"/>
 	<xacro:property name="joint_damping" value="0.0"/>
 	<xacro:property name="joint_friction" value="0.0"/>
@@ -46,4 +46,7 @@
 	<!-- ONLY USING COLLISION MESHES FOR INITIAL TESTING -->
 	<!-- REMEMBER TO ADD VISUAL/COLLISION MESHES!!!!~ -->
+		<!--############-->
+		<!-- LINK LINKS -->
+		<!--############-->
 		<link name="${prefix}link1">
 			<xacro:link_inertial ixx="0.0001" iyy="0.0001" izz="0.0001"/>
@@ -91,5 +94,7 @@
 			</collision>
 		</link>
+		<!--############-->
 		<!-- DISK LINKS -->
+		<!--############-->
 		<link name="base_link"/>
 		<link name="${prefix}disk1">
@@ -138,5 +143,8 @@
 			</collision>
 		</link>
-		<!-- END EFFECTOR
+		<!--##############-->
+		<!-- END EFFECTOR -->
+		<!--##############-->
+		<link name="${prefix}virtual_primary_link"/>
 		<link name="${prefix}end_effector">
 			<inertial>
@@ -152,5 +160,5 @@
 					<mesh filename="file://$(find spm_description)/meshes/end_effector_collision.stl"/>
 				</geometry>
-				<origin xyz="0.0 0.0 0.0" rpy="0.0 0.0 0.0"/>
+				<origin xyz="0.049496 0.0 0.039663" rpy="0.0 ${-pi/3} 0.0"/>
 			</visual>
 			<collision>
@@ -158,9 +166,10 @@
 					<mesh filename="file://$(find spm_description)/meshes/end_effector_collision.stl"/>
 				</geometry>
-				<origin xyz="0.0 0.0 0.0" rpy="0.0 0.0 0.0"/>
-			</collision>
-		</link>
-		-->
+				<origin xyz="0.049496 0.0 0.039663" rpy="0.0 ${-pi/3} 0.0"/>
+			</collision>
+		</link>
+		<!--#####################-->
 		<!-- BASE TO DISK JOINTS -->
+		<!--#####################-->
 		<joint name="${prefix}disk1_to_base" type="continuous">
 			<axis xyz="0.0 0.0 1.0"/>
@@ -187,5 +196,7 @@
 			<dynamics damping="${joint_damping}" friction="${joint_friction}"/>
 		</joint>
+		<!--#####################-->
 		<!-- DISK TO LINK JOINTS -->
+		<!--#####################-->
 		<joint name="${prefix}link1_to_disk1" type="continuous">
 			<axis xyz="0.0 0.0 1.0"/>
@@ -212,5 +223,20 @@
 			<dynamics damping="${joint_damping}" friction="${joint_friction}"/>
 		</joint>
+		<!--#############################-->
 		<!-- LINK TO END EFFECTOR JOINTS -->
+		<!--#############################-->
+		<joint name="${prefix}primary_joint_ref" type="fixed">
+			<parent link="${prefix}link1"/>
+			<child link="${prefix}virtual_primary_link"/>
+			<origin xyz="0.0 0.0 0.0" rpy="${-pi/4} 0.0 0.0"/>
+		</joint>
+		<joint name="${prefix}end_effector1_to_link1" type="continuous">
+			<axis xyz="0.0 0.0 1.0"/>
+			<limit effort="${joint_effort}" velocity="${joint_velocity}"/>
+			<parent link="${prefix}virtual_primary_link"/>
+			<child link="${prefix}end_effector"/>
+			<origin xyz="-0.059097 -0.060411 0.026633" rpy="0.0 ${pi/3} 0.0"/>
+			<dynamics damping="${joint_damping}" friction="${joint_friction}"/>
+		</joint>
 	</xacro:macro>
 </robot>

Commit message: generate sdf for gazebo

File: src/spm_sim_stack/spm_description/urdf/robots/spm_mechanism.urdf.xacro (robot description, xacro)
@@ -32,4 +32,14 @@
 		</inertial>
 	</xacro:macro>
+	<xacro:macro name="virtual_link_inertial">
+		<inertial>
+			<origin xyz="0.0 0.0 0.0" rpy="0.0 0.0 0.0"/>
+			<mass value="0.001"/>
+			<inertia
+			ixx="0.01" ixy="0.0" ixz="0.0"
+			iyy="0.01" iyz="0.0"
+			izz="0.01"/>
+		</inertial>
+	</xacro:macro>
 	<xacro:macro name="material_collision" params="ref_link ambient diffuse specular">
 		<gazebo reference="${ref_link}">
@@ -97,5 +107,7 @@
 		<!-- DISK LINKS -->
 		<!--############-->
-		<link name="base_link"/>
+		<link name="base_link">
+			<xacro:virtual_link_inertial/>
+		</link>
 		<link name="${prefix}disk1">
 			<xacro:disk_inertial mass="${disk1_mass}" ixx="0.0001" iyy="0.0001" izz="0.0001"/>
@@ -146,5 +158,13 @@
 		<!-- END EFFECTOR -->
 		<!--##############-->
-		<link name="${prefix}virtual_primary_link"/>
+		<link name="${prefix}virtual_primary_link">
+			<xacro:virtual_link_inertial/>
+		</link>
+		<link name="${prefix}virtual_link2">
+			<xacro:virtual_link_inertial/>
+		</link>
+		<link name="${prefix}virtual_link3">
+			<xacro:virtual_link_inertial/>
+		</link>
 		<link name="${prefix}end_effector">
 			<inertial>
@@ -231,4 +251,7 @@
 			<origin xyz="0.0 0.0 0.0" rpy="${-pi/4} 0.0 0.0"/>
 		</joint>
+		<joint name="${prefix}virtual_joint2" type="fixed">
+			<parent link="${prefix}end_effector"/>
+			<child link="${prefix}virtual_link2"/>
 		<joint name="${prefix}end_effector1_to_link1" type="continuous">
 			<axis xyz="0.0 0.0 1.0"/>
@@ -239,4 +262,14 @@
 			<dynamics damping="${joint_damping}" friction="${joint_friction}"/>
 		</joint>
+		<!--
+		<gazebo>
+			<joint name="${prefix}end_effector2_to_link2" type="continuous">
+				<parent>link2</parent>
+				<child>end_effector</child>
+				<pose>0 0 0 0 0 0</pose>
+				<axis><xyz>0 0 1</xyz></axis>
+			</joint>
+		</gazebo>
+				-->
 	</xacro:macro>
 </robot>
